File: hardware/serial-character-display/serial-character-display.kicad_sch (KiCad schematic)
At the start: 4 parts, among them SW1 SW_DIP_x01, U1 rp2040-zero

Commit message: add missing connection
Connections:
- net at DS1.2 (VDD), R1.1, U1.23 (5V): now also DS1.3 (VO)
Changed lines of the file:
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@@
 	(paper "A4")
+	(junction
+		(at 215.9 69.85)
+		(diameter 0)
+		(color 0 0 0 0)
+	)
 	(junction
 		(at 201.93 69.85)
@@
 	(wire
 		(pts
+			(xy 215.9 80.01) (xy 215.9 69.85)
+		)
+		(stroke
+			(width 0)
+			(type default)
+		)
+	)
+	(wire
+		(pts
 			(xy 152.4 92.71) (xy 140.97 92.71)
 		)
@@
 	(wire
 		(pts
+			(xy 212.09 80.01) (xy 215.9 80.01)
+		)
+		(stroke
+			(width 0)
+			(type default)
+		)
+	)
+	(wire
+		(pts
 			(xy 191.77 82.55) (xy 190.5 82.55)
 		)
@@
 	(wire
 		(pts
+			(xy 215.9 69.85) (xy 223.52 69.85)
+		)
+		(stroke
+			(width 0)
+			(type default)
+		)
+	)
+	(wire
+		(pts
 			(xy 185.42 121.92) (xy 148.59 121.92)
 		)
@@
 	(wire
 		(pts
-			(xy 201.93 69.85) (xy 223.52 69.85)
-		)
-		(stroke
+			(xy 201.93 69.85) (xy 215.9 69.85)
+		)
+		(stroke
